File: USB2514B_USB_Hub.kicad_sch (KiCad schematic)
At the start: 65 parts, among them J2 5V, J3 5V_OUT, Q1 40p04, U11 AP2141WG, U14 USB2514B_Bi, U15 USBLC6-2SC6, U16 USBLC6-2SC6, U17 USBLC6-2SC6, U18 USBLC6-2SC6, U2 AP2141WG, U3 AP2141WG, U4 AP2141WG, Y2 24MHz

Commit message: new file:   USB2514B_USB_Hub-backups/USB2514B_USB_Hub-2026-01-04_103254.zip 	new file:   USB2514B_USB_Hub-backups/USB2514B_USB_Hub-2026-01-04_104353.zip 	new file:   USB2514B_USB_Hub-backups/USB2514B_USB_Hub-2026-01-04_104902.zip 	modified:   USB2514B_USB_Hub.kicad_pro 	modified:   USB2514B_USB_Hub.kicad_sch 	new file:   untitled.kicad_sch 	deleted:    ~USB2514B_USB_Hub.kicad_sch.lck
Parts:
- removed C14, C15, C16, C17, C18, C19, C3, C4, C57: 2.2uF, Capacitor_SMD:C_0603_1608Metric_Pad1.08x0.95mm_HandSolder, symbol Device:C_Small
- removed F1: 500mA, Fuse:Fuse_0805_2012Metric, symbol Device:Polyfuse_Small
- removed FB1: 120R, Inductor_SMD:L_0603_1608Metric_Pad1.05x0.95mm_HandSolder, symbol Device:FerriteBead_Small
- removed R44, R45, R46, R47, R52, R53: 5.1k_1%, Resistor_SMD:R_0603_1608Metric_Pad0.98x0.95mm_HandSolder, symbol Device:R_Small
- removed U11, U2, U3, U4: AP2141WG, Package_TO_SOT_SMD:SOT-23-5_HandSoldering, symbol Power_Management:AP2161W
- removed U15, U16, U17, U18: USBLC6-2SC6, Package_TO_SOT_SMD:SOT-23-6, symbol Power_Protection:USBLC6-2SC6
- removed USB1, USB2, USB3: USB_C_Recep._USB2.0_16P, Connector_USB:USB_C_Receptacle_GCT_USB4105-xx-A_16P_TopMnt_Horizontal, symbol Connector:USB_C_Receptacle_USB2.0_16P
- removed USB4: USB_A, My_Library:USB_A_2.0, symbol Connector:USB_A
- renumbered C6 to C1, C58 to C10, C44 to C11, C45 to C12, C46 to C13, C47 to C14, C48 to C15, C49 to C16, C5 to C2, C50 to C3, C51 to C4, C52 to C5, C53 to C6, C54 to C7, C55 to C8, C56 to C9, D8 to D1, D7 to D2, F2 to F1, J2 to J1, J3 to J2, R0_2 to R0_1, R26 to R1, R48 to R10, R38 to R2, R39 to R3, R40 to R4, R41 to R5, R51 to R6, R50 to R7, R43 to R8, R42 to R9, U14 to U1, Y2 to Y1
Connections:
- net USB_STM_D+ renamed USB_HUB_1D+
- net USB_STM_D- renamed USB_HUB_1D-
- no-connect marks 6 -> 0
Other:
- added sheet Sheet_2 (untitled.kicad_sch)
- note removed: "Resistors are integrated into the chip"
- note removed: "USB In"
- note removed: "USB Out 2"
- note removed: "USB Out 3"
- note removed: "USB Out 4"
- moved on the sheet: C1, C10, C11, C12, C13, C14, C15, C16, C2, C3, C4, C5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
